File: Optokoppler_Tester.kicad_sch (KiCad schematic)
At the start: 17 parts, among them J1 USB_C_Receptacle_USB2.0, SW1 SW_Push, U1 LTV-847M

Commit message: Added versioning
Other:
- company: (none) -> André Fiedler <mail@andrefiedler.de>
- title: (none) -> Optokoppler Tester
Changed lines of the file:
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@@
 	(generator_version "9.0")
 	(paper "A4")
+	(title_block
+		(title "Optokoppler Tester")
+		(date "2025-07-20")
+		(rev "v1.0")
+		(company "André Fiedler <mail@andrefiedler.de>")
+	)
 	(junction
 		(at 264.16 31.75)
